Commit message: changes corresponding to xacros

File: catkin_ws/src/my_robot/urdf/my_robot.xacro (robot description, xacro)
@@ -2,4 +2,5 @@
 <robot name="my_robot" xmlns:xacro="http://www.ros.org/wiki/xacro">
 <xacro:include filename="materials.xacro"/>
+<xacro:include filename="$(find my_robot)/urdf/my_robot.gazebo" />
 <link name="robot_footprint"></link>
 <joint name="robot_footprint_joint" type="fixed">
@@ -143,7 +144,7 @@
       <box size="0.05 0.05 0.05"/>
     </geometry>
-    <material name="BlueMaterial">
-      <xacro:BlueMaterial/>
-    </material>
+    <gazebo reference="camera">
+    <material>Gazebo/Green</material>
+    </gazebo>
   </visual>
 </link>
