Commit message: replaced my robot with latest changes

File: src/my_robot/urdf/materials.xacro (robot description, xacro)
@@ -3,5 +3,8 @@
   <xacro:macro name="BlueMaterial" params="">
     <material name="Blue">
-      <color rgba="0 0 1 1"/>
+      <ambient>0 0 1 1</ambient>
+      <diffuse>0 0 1 1</diffuse>
+      <specular>0.1 0.1 0.1 1</specular>
+      <emissive>0 0 0 1</emissive>
     </material>
   </xacro:macro>

File: src/my_robot/urdf/my_robot.xacro (robot description, xacro)
@@ -2,4 +2,5 @@
 <robot name="my_robot" xmlns:xacro="http://www.ros.org/wiki/xacro">
 <xacro:include filename="materials.xacro"/>
+<xacro:include filename="$(find my_robot)/urdf/my_robot.gazebo" />
 <link name="robot_footprint"></link>
 <joint name="robot_footprint_joint" type="fixed">
@@ -30,4 +31,7 @@
       <box size=".4 .2 .1"/>
     </geometry>
+    <material name="BlueMaterial">
+      <xacro:BlueMaterial/>
+    </material>
   </visual>
   <collision name='back_caster_collision'>
@@ -140,7 +144,7 @@
       <box size="0.05 0.05 0.05"/>
     </geometry>
-    <material name="Blue">
-      <xacro:BlueMaterial/>
-    </material>
+    <gazebo reference="camera">
+    <material>Gazebo/Green</material>
+    </gazebo>
   </visual>
 </link>

Commit message: material bug fixed

File: src/my_robot/urdf/materials.xacro (robot description, xacro)
@@ -9,3 +9,6 @@
     </material>
   </xacro:macro>
+<gazebo reference="chassis">
+    <material>Gazebo/Blue</material>
+  </gazebo>
 </robot>

File: src/my_robot/urdf/my_robot.xacro (robot description, xacro)
@@ -31,8 +31,8 @@
       <box size=".4 .2 .1"/>
     </geometry>
-    <material name="BlueMaterial">
-      <xacro:BlueMaterial/>
-    </material>
   </visual>
+<gazebo reference="chassis">
+  <material>Gazebo/Blue</material>
+</gazebo>
   <collision name='back_caster_collision'>
     <origin xyz="-0.15 0 -0.05" rpy="0 0 0"/>
@@ -144,9 +144,9 @@
       <box size="0.05 0.05 0.05"/>
     </geometry>
-    <gazebo reference="camera">
-    <material>Gazebo/Green</material>
-    </gazebo>
   </visual>
 </link>
+<gazebo reference="camera">
+   <material>Gazebo/Green</material>
+</gazebo>
 <joint type="fixed" name="camera_joint">
     <origin xyz="0.2 0 0" rpy="0 0 0"/>

Commit message: fixes after comments on project

File: src/my_robot/urdf/materials.xacro (robot description, xacro)
@@ -10,5 +10,5 @@
   </xacro:macro>
 <gazebo reference="chassis">
-    <material>Gazebo/Blue</material>
+    <material>Gazebo/Red</material>
   </gazebo>
 </robot>

File: src/my_robot/urdf/my_robot.xacro (robot description, xacro)
@@ -33,5 +33,5 @@
   </visual>
 <gazebo reference="chassis">
-  <material>Gazebo/Blue</material>
+  <material>Gazebo/Red</material>
 </gazebo>
   <collision name='back_caster_collision'>
