Commit message: robot enhancements done

File: src/my_robot/urdf/my_robot.xacro (robot description, xacro)
@@ -11,5 +11,5 @@
   <inertial>
     <mass value="15.0"/>
-    <origin xyz="0.0 0 0" rpy=" 0 0 0"/>
+    <origin xyz="0.0 0 0" rpy="0 0 0"/>
     <inertia
         ixx="0.1" ixy="0" ixz="0"
@@ -18,6 +18,6 @@
     />
   </inertial>
-  <collision name='collision'>
-    <origin xyz="0 0 0" rpy=" 0 0 0"/>
+  <collision name='chassis_collision'>
+    <origin xyz="0 0 0" rpy="0 0 0"/>
     <geometry>
       <box size=".4 .2 .1"/>
@@ -25,5 +25,5 @@
   </collision>
   <visual name='chassis_visual'>
-    <origin xyz="0 0 0" rpy=" 0 0 0"/>
+    <origin xyz="0 0 0" rpy="0 0 0"/>
     <geometry>
       <box size=".4 .2 .1"/>
@@ -31,5 +31,5 @@
   </visual>
   <collision name='back_caster_collision'>
-    <origin xyz="-0.15 0 -0.05" rpy=" 0 0 0"/>
+    <origin xyz="-0.15 0 -0.05" rpy="0 0 0"/>
     <geometry>
       <sphere radius="0.0499"/>
@@ -55,8 +55,8 @@
   </visual>
 </link>
-<link name='SIDE_wheel'>
+<link name='left_wheel'>
 <inertial>
-    <mass value="15.0"/>
-    <origin xyz="0.0 0 0" rpy=" 0 0 0"/>
+    <mass value="5.0"/>
+    <origin xyz="0.0 0 0" rpy=" 0 1.5707 1.5707"/>
     <inertia
         ixx="0.1" ixy="0" ixz="0"
@@ -65,16 +65,114 @@
     />
   </inertial>
-  <collision name='collision'>
-    <origin xyz="0 0 0" rpy=" 0 0 0"/>
+  <collision name='left_wheel_collision'>
+    <origin xyz="0.0 0 0" rpy=" 0 1.5707 1.5707"/>
     <geometry>
-      <box size=".4 .2 .1"/>
+      <cylinder radius="0.1" length="0.05"/>
     </geometry>
   </collision>
-  <visual name='chassis_visual'>
-    <origin xyz="0 0 0" rpy=" 0 0 0"/>
+  <visual name='left_wheel_visual'>
+    <origin xyz="0 0 0" rpy=" 0 1.5707 1.5707"/>
     <geometry>
-      <box size=".4 .2 .1"/>
+      <cylinder radius="0.1" length="0.05"/>
     </geometry>
   </visual>
 </link>
+<joint type="continuous" name="left_wheel_hinge">
+    <origin xyz="0 0.15 0" rpy="0 0 0"/>
+    <child link="left_wheel"/>
+    <parent link="chassis"/>
+    <axis xyz="0 1 0" rpy="0 0 0"/>
+    <limit effort="10000" velocity="1000"/>
+    <dynamics damping="1.0" friction="1.0"/>
+  </joint>
+<link name='right_wheel'>
+<inertial>
+    <mass value="5.0"/>
+    <origin xyz="0 0 0" rpy=" 0 1.5707 1.5707"/>
+    <inertia
+        ixx="0.1" ixy="0" ixz="0"
+        iyy="0.1" iyz="0"
+        izz="0.1"
+    />
+  </inertial>
+  <collision name='right_wheel_collision'>
+    <origin xyz="0.0 0 0" rpy=" 0 1.5707 1.5707"/>
+    <geometry>
+      <cylinder radius="0.1" length="0.05"/>
+    </geometry>
+  </collision>
+  <visual name='right_wheel_visual'>
+    <origin xyz="0 0 0" rpy=" 0 1.5707 1.5707"/>
+    <geometry>
+      <cylinder radius="0.1" length="0.05"/>
+    </geometry>
+  </visual>
+</link>
+<joint type="continuous" name="right_wheel_hinge">
+    <origin xyz="0 -0.15 0" rpy="0 0 0"/>
+    <child link="right_wheel"/>
+    <parent link="chassis"/>
+    <axis xyz="0 1 0" rpy="0 0 0"/>
+    <limit effort="10000" velocity="1000"/>
+    <dynamics damping="1.0" friction="1.0"/>
+  </joint>
+<!-- Camera link and joint added -->
+<link name="camera">
+  <inertial>
+     <mass value="0.1"/>
+     <origin xyz="0 0 0" rpy="0 0 0"/>
+     <inertia
+       ixx="1e-6" ixy="0" ixz="0"
+       iyy="1e-6" iyz="0"
+       izz="1e-6"
+     />
+  </inertial>
+  <collision name="camera_collision">
+    <origin xyz="0 0 0" rpy="0 0 0"/>
+    <geometry>
+      <box size="0.05 0.05 0.05"/>
+    </geometry>
+  </collision>
+  <visual name="camera_visual">
+    <origin xyz="0 0 0" rpy="0 0 0"/>
+    <geometry>
+      <box size="0.05 0.05 0.05"/>
+    </geometry>
+  </visual>
+</link>
+<joint type="fixed" name="camera_joint">
+    <origin xyz="0.2 0 0" rpy="0 0 0"/>
+    <child link="camera"/>
+    <parent link="chassis"/>
+  </joint>
+<!-- Lidar Link and joint -->
+<link name="hokuyo">
+   <inertial>
+     <mass value="1e-6"/>
+     <origin xyz="0 0 0" rpy="0 0 0"/>
+     <inertia
+       ixx="1e-6" ixy="0" ixz="0"
+       iyy="1e-6" iyz="0"
+       izz="1e-6"
+     />
+   </inertial>
+   <collision name="hokuyo_collision">
+     <origin xyz="0 0 0" rpy="0 0 0"/>
+     <geometry>
+       <box size="0.1 0.1 0.1"/>
+     </geometry>
+   </collision>
+   <visual name="hokuyo_visual">
+      <origin xyz="0 0 0" rpy="0 0 0"/>
+     <geometry>
+       <mesh filename="package://my_robot/meshes/hokuyo.dae" scale="1 1 1"/>
+     </geometry>
+   </visual>
+</link>
+<joint type="fixed" name="hokuyo_joint">
+    <origin xyz="0.15 0 0.1" rpy="0 0 0"/>
+    <child link="hokuyo"/>
+    <parent link="chassis"/>
+    <axis xyz="0 1 0"/>
+</joint>
 </robot>

Commit message: Added materials.xacro

File: src/my_robot/urdf/my_robot.xacro (robot description, xacro)
@@ -1,4 +1,5 @@
 <?xml version='1.0'?>
 <robot name="my_robot" xmlns:xacro="http://www.ros.org/wiki/xacro">
+<xacro:include filename="materials.xacro"/>
 <link name="robot_footprint"></link>
 <joint name="robot_footprint_joint" type="fixed">
@@ -139,4 +140,7 @@
       <box size="0.05 0.05 0.05"/>
     </geometry>
+    <material name="Blue">
+      <xacro:BlueMaterial/>
+    </material>
   </visual>
 </link>

Commit message: added materials and topics verified

File: src/my_robot/urdf/my_robot.xacro (robot description, xacro)
@@ -83,4 +83,7 @@
   </visual>
 </link>
+<gazebo reference="left_wheel">
+   <material>Gazebo/Black</material>
+</gazebo>
 <joint type="continuous" name="left_wheel_hinge">
     <origin xyz="0 0.15 0" rpy="0 0 0"/>
@@ -114,4 +117,7 @@
   </visual>
 </link>
+<gazebo reference="right_wheel">
+   <material>Gazebo/Black</material>
+</gazebo>
 <joint type="continuous" name="right_wheel_hinge">
     <origin xyz="0 -0.15 0" rpy="0 0 0"/>

Commit message: changed chassis dimensions & wheel radius

File: src/my_robot/urdf/my_robot.xacro (robot description, xacro)
@@ -23,5 +23,5 @@
     <origin xyz="0 0 0" rpy="0 0 0"/>
     <geometry>
-      <box size=".4 .2 .1"/>
+      <box size=".4 .2 .08"/>
     </geometry>
   </collision>
@@ -29,5 +29,5 @@
     <origin xyz="0 0 0" rpy="0 0 0"/>
     <geometry>
-      <box size=".4 .2 .1"/>
+      <box size=".4 .2 .08"/>
     </geometry>
   </visual>
@@ -36,5 +36,5 @@
 </gazebo>
   <collision name='back_caster_collision'>
-    <origin xyz="-0.15 0 -0.05" rpy="0 0 0"/>
+    <origin xyz="-0.10 0 -0.05" rpy="0 0 0"/>
     <geometry>
       <sphere radius="0.0499"/>
@@ -42,5 +42,5 @@
   </collision>
   <visual name='back_caster_visual'>
-    <origin xyz="-0.15 0 -0.05" rpy=" 0 0 0"/>
+    <origin xyz="-0.10 0 -0.05" rpy=" 0 0 0"/>
     <geometry>
       <sphere radius="0.05"/>
@@ -48,5 +48,5 @@
   </visual>
   <collision name='front_caster_collision'>
-    <origin xyz="0.15 0 -0.05" rpy=" 0 0 0"/>
+    <origin xyz="0.10 0 -0.05" rpy=" 0 0 0"/>
     <geometry>
       <sphere radius="0.0499"/>
@@ -54,5 +54,5 @@
   </collision>
   <visual name='front_caster_visual'>
-    <origin xyz="0.15 0 -0.05" rpy=" 0 0 0"/>
+    <origin xyz="0.10 0 -0.05" rpy=" 0 0 0"/>
     <geometry>
       <sphere radius="0.05"/>

Commit message: fixed sunken robot issue

File: src/my_robot/urdf/my_robot.xacro (robot description, xacro)
@@ -5,5 +5,5 @@
 <link name="robot_footprint"></link>
 <joint name="robot_footprint_joint" type="fixed">
-  <origin xyz="0 0 0" rpy="0 0 0" />
+  <origin xyz="0 0 0.1" rpy="0 0 0" />
   <parent link="robot_footprint"/>
   <child link="chassis" />

Commit message: mapping launch file added

File: src/my_robot/urdf/my_robot.xacro (robot description, xacro)
@@ -154,4 +154,11 @@
   </visual>
 </link>
+  <joint name="camera_optical_joint" type="fixed">
+    <origin xyz="0 0 0" rpy="-1.5707 0 -1.5707"/>
+    <parent link="camera"/>
+    <child link="camera_link_optical"/>
+  </joint>
+  <link name="camera_link_optical">
+  </link>
 <gazebo reference="camera">
    <material>Gazebo/Green</material>

Commit message: camera topic is the issue

File: src/my_robot/urdf/my_robot.xacro (robot description, xacro)
@@ -154,4 +154,13 @@
   </visual>
 </link>
+<gazebo reference="camera">
+   <material>Gazebo/Green</material>
+</gazebo>
+<joint type="fixed" name="camera_joint">
+    <origin xyz="0.2 0 0" rpy="0 0 0"/>
+    <child link="camera"/>
+    <parent link="chassis"/>
+    <imageTopicName>rgb/image_raw</imageTopicName>
+  </joint>
   <joint name="camera_optical_joint" type="fixed">
     <origin xyz="0 0 0" rpy="-1.5707 0 -1.5707"/>
@@ -161,13 +170,4 @@
   <link name="camera_link_optical">
   </link>
-<gazebo reference="camera">
-   <material>Gazebo/Green</material>
-</gazebo>
-<joint type="fixed" name="camera_joint">
-    <origin xyz="0.2 0 0" rpy="0 0 0"/>
-    <child link="camera"/>
-    <parent link="chassis"/>
-    <imageTopicName>rgb/image_raw</imageTopicName>
-  </joint>
 <!-- Lidar Link and joint -->
 <link name="hokuyo">
